Commit message: Remove unnecessary staff

File: drone/drone_description/urdf/italdron_evo4hse.urdf.xacro (robot description, xacro)
@@ -2,4 +2,5 @@
 <robot name="quadrotor" xmlns:xacro="http://www.ros.org/wiki/xacro">
     <xacro:property name="M_PI" value="3.1415926535897931" />
+    <xacro:include filename="$(find drone_gazebo)/urdf/quadrotor_plugins.gazebo.xacro" />
     <!-- Included URDF Files -->
     <!-- The base includes a hokuyo lidar used for height estimation -->

File: drone/drone_description/urdf/quadrotor_custom_base.urdf.xacro (robot description, xacro)
@@ -27,4 +27,6 @@
       <origin xyz="0.0 0.0 -0.065" rpy="0.0 0 0"/>
     </xacro:lightware_sf11_120m>
+    <!-- Gazebo Plugins -->
+    <xacro:quadrotor_plugins/>
   </xacro:macro>
 </robot>

File: drone/drone_gazebo/urdf/quadrotor_plugins.gazebo.xacro (robot description, xacro)
@@ -8,7 +8,10 @@
   <xacro:include filename="$(find drone_gazebo)/urdf/quadrotor_aerodynamics.gazebo.xacro" />
   <!-- Quadrotor Gazebo Plugins -->
-  <xacro:quadrotor_sensors />
-  <xacro:quadrotor_controller />
-  <xacro:quadrotor_propulsion />
-  <xacro:quadrotor_aerodynamics />
+  <xacro:macro name="quadrotor_plugins">
+    <canonicalBody>base_link</canonicalBody>
+    <xacro:quadrotor_sensors/>
+    <xacro:quadrotor_controller />
+    <xacro:quadrotor_propulsion />
+    <xacro:quadrotor_aerodynamics />
+  </xacro:macro>
 </robot>

File: drone/drone_gazebo/urdf/quadrotor_sensors.gazebo.xacro (robot description, xacro)
@@ -4,57 +4,4 @@
   <xacro:macro name="quadrotor_sensors">
         <gazebo>
-    <!--
-          <plugin name="quadrotor_imu_sim" filename="libhector_gazebo_ros_imu.so">
-            <updateRate>100.0</updateRate>
-            <bodyName>base_link</bodyName>
-            <frameId>$(arg base_link_frame)</frameId>
-            <topicName>raw_imu</topicName>
-            <rpyOffset>0 0 0</rpyOffset>
-            <gaussianNoise>0</gaussianNoise>
-            <accelDrift>0.1 0.1 0.1</accelDrift>
-            <accelGaussianNoise>0.35 0.35 0.3</accelGaussianNoise>
-            <rateDrift>0.1 0.1 0.1</rateDrift>
-            <rateGaussianNoise>0.05 0.05 0.015</rateGaussianNoise>
-          </plugin>
-          <plugin name="quadrotor_baro_sim" filename="libhector_gazebo_ros_baro.so">
-            <updateRate>10.0</updateRate>
-            <bodyName>base_link</bodyName>
-            <frameId>$(arg base_link_frame)</frameId>
-            <topicName>pressure_height</topicName>
-            <altimeterTopicName>altimeter</altimeterTopicName>
-            <offset>0</offset>
-            <drift>10.0</drift>
-            <gaussianNoise>0.1</gaussianNoise>
-          </plugin>
-          <plugin name="quadrotor_magnetic_sim" filename="libhector_gazebo_ros_magnetic.so">
-            <updateRate>10.0</updateRate>
-            <bodyName>base_link</bodyName>
-            <frameId>$(arg base_link_frame)</frameId>
-            <topicName>magnetic</topicName>
-            <offset>0 0 0</offset>
-            <drift>0.0 0.0 0.0</drift>
-            <gaussianNoise>1.3e-2 1.3e-2 1.3e-2</gaussianNoise>
-          </plugin>
-          <plugin name="quadrotor_gps_sim" filename="libhector_gazebo_ros_gps.so">
-            <updateRate>4.0</updateRate>
-            <bodyName>base_link</bodyName>
-            <frameId>$(arg base_link_frame)</frameId>
-            <topicName>fix</topicName>
-            <velocityTopicName>fix_velocity</velocityTopicName>
-            <referenceLatitude>49.860246</referenceLatitude>
-            <referenceLongitude>8.687077</referenceLongitude>
-            <drift>5.0 5.0 5.0</drift>
-            <gaussianNoise>0.01 0.01 0.01</gaussianNoise>
-            <velocityDrift>0 0 0</velocityDrift>
-            <velocityGaussianNoise>0.05 0.05 0.05</velocityGaussianNoise>
-          </plugin>
-          <plugin name="quadrotor_groundtruth_sim" filename="libgazebo_ros_p3d.so">
-            <updateRate>100.0</updateRate>
-            <bodyName>base_link</bodyName>
-            <topicName>ground_truth/state</topicName>
-            <gaussianNoise>0.0</gaussianNoise>
-            <frameName>$(arg world_frame)</frameName>
-          </plugin>
--->
           <plugin name="p3d_base_controller" filename="libgazebo_ros_p3d.so">
             <alwaysOn>true</alwaysOn>

Commit message: Add TF listener for height receiver

File: drone/drone_description/urdf/italdron_evo4hse.urdf.xacro (robot description, xacro)
@@ -16,3 +16,8 @@
     <origin xyz="0.125 0 -0.17" rpy="0 0 0"/>
     </xacro:generic_camera>
+    <!-- LightWare SF11 (120 meter) height sensor -->
+    <xacro:include filename="$(find drone_description)/sensors/lightware_sf11_120m.urdf.xacro" />
+    <xacro:lightware_sf11_120m name="height_sensor" parent="base_link" ros_topic="lidar/height/scan" update_rate="100" ray_count="5" min_angle="-87" max_angle="-93" >
+      <origin xyz="0.0 0.0 0" rpy="0.0 0 0"/>
+    </xacro:lightware_sf11_120m>
 </robot>

File: drone/drone_description/urdf/quadrotor_custom_base.urdf.xacro (robot description, xacro)
@@ -1,5 +1,4 @@
 <?xml version="1.0"?>
 <robot xmlns:xacro="http://www.ros.org/wiki/xacro">
-  <xacro:include filename="$(find drone_description)/sensors/lightware_sf11_120m.urdf.xacro" />
   <!-- Main quadrotor link -->
   <xacro:macro name="quadrotor_base_macro">
@@ -23,8 +22,4 @@
       </collision>
     </link>
-    <!-- LightWare SF11 (120 meter) height sensor -->
-    <xacro:lightware_sf11_120m name="height_sensor" parent="base_link" ros_topic="lidar/height/scan" update_rate="100" ray_count="5" min_angle="-87" max_angle="-93" >
-      <origin xyz="0.0 0.0 -0.065" rpy="0.0 0 0"/>
-    </xacro:lightware_sf11_120m>
     <!-- Gazebo Plugins -->
     <xacro:quadrotor_plugins/>
